File: hardware/temp_sensor_ring/temp_sens_ring.sch (EAGLE design)
At the start: 13 parts, among them IC1 MCP9808

Commit message: inital board commit
Parts:
- removed JP1: A0, SparkFun-Jumpers:JUMPER-SMT_3_NO_SILK
- removed JP2: A1, SparkFun-Jumpers:JUMPER-SMT_3_NO_SILK
- removed JP3: A2, SparkFun-Jumpers:JUMPER-SMT_3_NO_SILK
- added J1, J2, J3: (no value), SIG_Parts:SMD_JUMP_2_NO_S
- added R2: (no value), SIG_Parts:RESISTOR_NET_4-0502
Connections:
- removed net N$16: X1G$1.8
- removed net N$7: X2G$1.8
- net +3V3: now also J1.2, J2.2, J3.2, X1G$1.8, X2G$1.8; no longer JP1.3, JP2.3, JP3.3
- net GND: now also R2-1.2, R2-2.2, R2-3.2, R2-4.2; no longer JP1.1, JP2.1, JP3.1
- net N$1: now also J3.1, R2-3.1; no longer JP3.2
- net N$2: now also J1.1, R2-2.1; no longer JP2.2
- net N$3: now also J2.1, R2-1.1; no longer JP1.2

Commit message: PCB completed, part library created
Connections:
- net GND: now also R2-1.1, R2-2.1, R2-3.1, R2-4.1; no longer R2-1.2, R2-2.2, R2-3.2, R2-4.2
- net N$1: now also R2-2.2; no longer R2-3.1
- net N$2: now also R2-3.2; no longer R2-2.1
- net N$3: now also R2-4.2; no longer R2-1.1
Other:
- moved on the sheet: R2-1, R2-2, R2-3, R2-4
Changed lines of the file:
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@@
 <part name="J1" library="SIG_Parts" deviceset="SMD_JUMP_2_NO_" device="S"/>
 <part name="J3" library="SIG_Parts" deviceset="SMD_JUMP_2_NO_" device="S"/>
+<part name="GND10" library="supply1" library_urn="urn:adsk.eagle:library:371" deviceset="GND" device=""/>
 <part name="R2" library="SIG_Parts" deviceset="RESISTOR_NET_*" device="4-0502"/>
-<part name="GND10" library="supply1" library_urn="urn:adsk.eagle:library:371" deviceset="GND" device=""/>
+<part name="FRAME1" library="SIG_Parts" deviceset="FRAME_A4_FULL" device=""/>
 </parts>
 <sheets>
@@
 <attribute name="VALUE" x="17.78" y="40.64" size="1.778" layer="96" font="vector" rot="R180" align="top-left"/>
 </instance>
-<instance part="R2" gate="-1" x="43.18" y="25.4" smashed="yes" rot="R270">
-<attribute name="NAME" x="44.6786" y="29.21" size="1.778" layer="95" rot="R270"/>
-<attribute name="VALUE" x="39.878" y="29.21" size="1.778" layer="96" rot="R270"/>
-</instance>
-<instance part="R2" gate="-2" x="33.02" y="25.4" smashed="yes" rot="R270">
-<attribute name="NAME" x="34.5186" y="29.21" size="1.778" layer="95" rot="R270"/>
-<attribute name="VALUE" x="29.718" y="29.21" size="1.778" layer="96" rot="R270"/>
-</instance>
-<instance part="R2" gate="-3" x="22.86" y="25.4" smashed="yes" rot="R270">
-<attribute name="NAME" x="24.3586" y="29.21" size="1.778" layer="95" rot="R270"/>
-<attribute name="VALUE" x="19.558" y="29.21" size="1.778" layer="96" rot="R270"/>
-</instance>
-<instance part="R2" gate="-4" x="12.7" y="25.4" smashed="yes" rot="R270">
-<attribute name="NAME" x="14.1986" y="29.21" size="1.778" layer="95" rot="R270"/>
-<attribute name="VALUE" x="9.398" y="29.21" size="1.778" layer="96" rot="R270"/>
-</instance>
 <instance part="GND10" gate="1" x="12.7" y="15.24" smashed="yes">
 <attribute name="VALUE" x="10.16" y="12.7" size="1.778" layer="96"/>
+</instance>
+<instance part="R2" gate="-1" x="12.7" y="25.4" smashed="yes" rot="R90">
+<attribute name="NAME" x="11.2014" y="21.59" size="1.778" layer="95" rot="R90"/>
+<attribute name="VALUE" x="16.002" y="21.59" size="1.778" layer="96" rot="R90"/>
+</instance>
+<instance part="R2" gate="-2" x="22.86" y="25.4" smashed="yes" rot="R90">
+<attribute name="NAME" x="21.3614" y="21.59" size="1.778" layer="95" rot="R90"/>
+<attribute name="VALUE" x="26.162" y="21.59" size="1.778" layer="96" rot="R90"/>
+</instance>
+<instance part="R2" gate="-3" x="33.02" y="25.4" smashed="yes" rot="R90">
+<attribute name="NAME" x="31.5214" y="21.59" size="1.778" layer="95" rot="R90"/>
+<attribute name="VALUE" x="36.322" y="21.59" size="1.778" layer="96" rot="R90"/>
+</instance>
+<instance part="R2" gate="-4" x="43.18" y="25.4" smashed="yes" rot="R90">
+<attribute name="NAME" x="41.6814" y="21.59" size="1.778" layer="95" rot="R90"/>
+<attribute name="VALUE" x="46.482" y="21.59" size="1.778" layer="96" rot="R90"/>
+</instance>
+<instance part="FRAME1" gate="G$1" x="-121.92" y="-83.82" smashed="yes">
+<attribute name="PROJECT_SECTION" x="93.98" y="-54.72" size="3" layer="97" font="vector" align="center"/>
+<attribute name="SHEET_NAME" x="94.18" y="-69.32" size="3" layer="97" font="vector" align="center"/>
+<attribute name="SHEET" x="145.58" y="-57.62" size="3" layer="97" font="vector" align="center"/>
+<attribute name="LARGE_NOTE" x="145.58" y="-70.32" size="3" layer="97" font="vector" align="center"/>
 </instance>
 </instances>
@@
 <wire x1="22.86" y1="38.1" x2="22.86" y2="30.48" width="0.1524" layer="91"/>
 <junction x="22.86" y="38.1"/>
-<pinref part="R2" gate="-3" pin="1"/>
+<pinref part="R2" gate="-2" pin="2"/>
 </segment>
 </net>
@@
 <wire x1="33.02" y1="45.72" x2="33.02" y2="30.48" width="0.1524" layer="91"/>
 <junction x="33.02" y="45.72"/>
-<pinref part="R2" gate="-2" pin="1"/>
+<pinref part="R2" gate="-3" pin="2"/>
 </segment>
 </net>
@@
 <wire x1="43.18" y1="53.34" x2="43.18" y2="30.48" width="0.1524" layer="91"/>
 <junction x="43.18" y="53.34"/>
-<pinref part="R2" gate="-1" pin="1"/>
+<pinref part="R2" gate="-4" pin="2"/>
 </segment>
 </net>
@@
 <pinref part="GND1" gate="1" pin="GND"/>
 <wire x1="22.86" y1="17.78" x2="22.86" y2="20.32" width="0.1524" layer="91"/>
-<pinref part="R2" gate="-3" pin="2"/>
+<pinref part="R2" gate="-2" pin="1"/>
 </segment>
 <segment>
 <pinref part="GND2" gate="1" pin="GND"/>
 <wire x1="33.02" y1="17.78" x2="33.02" y2="20.32" width="0.1524" layer="91"/>
-<pinref part="R2" gate="-2" pin="2"/>
+<pinref part="R2" gate="-3" pin="1"/>
 </segment>
 <segment>
 <pinref part="GND3" gate="1" pin="GND"/>
 <wire x1="43.18" y1="17.78" x2="43.18" y2="20.32" width="0.1524" layer="91"/>
-<pinref part="R2" gate="-1" pin="2"/>
+<pinref part="R2" gate="-4" pin="1"/>
 </segment>
 <segment>
 <wire x1="12.7" y1="20.32" x2="12.7" y2="17.78" width="0.1524" layer="91"/>
-<pinref part="R2" gate="-4" pin="2"/>
 <pinref part="GND10" gate="1" pin="GND"/>
-</segment>
-</net>
+<pinref part="R2" gate="-1" pin="1"/>
+</segment>
+</net>

Commit message: 3D models added to library
Parts:
- C1: device SIG_Parts:CAP_CERAMIC_0402 -> temp_sens_ring:CAP_CERAMIC_0402
- IC1: device SIG_Parts:MCP9808 -> temp_sens_ring:MCP9808
- J1, J2, J3: device SIG_Parts:SMD_JUMP_2_NO_S -> temp_sens_ring:SMD_JUMP_2_NO_S
- JP4, JP5, JP6, JP7, JP8: device SparkFun-Jumpers:JUMPER-SMT_2_NO_NO-SILK -> temp_sens_ring:JUMPER-SMT_2_NO_NO-SILK
- R1: device SIG_Parts:RESISTOR_0402 -> temp_sens_ring:RESISTOR_0402
- R2: device SIG_Parts:RESISTOR_NET_4-0502 -> temp_sens_ring:RESISTOR_NET_4-0502
- X1, X2: device SIG_Parts:FFC_10PV -> temp_sens_ring:FFC_10PV
Changed lines of the file:
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@@
 </classes>
 <parts>
-<part name="X1" library="SIG_Parts" deviceset="FFC_10P" device="V">
+<part name="X1" library="temp_sens_ring" library_urn="urn:adsk.eagle:library:31797301" deviceset="FFC_10P" device="V" package3d_urn="urn:adsk.eagle:package:31797271/2">
 <attribute name="MFR" value="XFCN"/>
 <attribute name="MFR_PART" value="F1002-B-10-20T-R"/>
 <attribute name="PITCH" value="1.00"/>
 </part>
-<part name="IC1" library="SIG_Parts" deviceset="MCP9808" device=""/>
-<part name="+3V1" library="supply1" library_urn="urn:adsk.eagle:library:371" deviceset="+3V3" device=""/>
-<part name="+3V2" library="supply1" library_urn="urn:adsk.eagle:library:371" deviceset="+3V3" device=""/>
-<part name="+3V3" library="supply1" library_urn="urn:adsk.eagle:library:371" deviceset="+3V3" device=""/>
-<part name="GND1" library="supply1" library_urn="urn:adsk.eagle:library:371" deviceset="GND" device=""/>
-<part name="GND2" library="supply1" library_urn="urn:adsk.eagle:library:371" deviceset="GND" device=""/>
-<part name="GND3" library="supply1" library_urn="urn:adsk.eagle:library:371" deviceset="GND" device=""/>
-<part name="GND4" library="supply1" library_urn="urn:adsk.eagle:library:371" deviceset="GND" device=""/>
-<part name="+3V4" library="supply1" library_urn="urn:adsk.eagle:library:371" deviceset="+3V3" device=""/>
-<part name="R1" library="SIG_Parts" deviceset="RESISTOR_*" device="0402" value="10K"/>
-<part name="+3V5" library="supply1" library_urn="urn:adsk.eagle:library:371" deviceset="+3V3" device=""/>
-<part name="GND5" library="supply1" library_urn="urn:adsk.eagle:library:371" deviceset="GND" device=""/>
-<part name="+3V6" library="supply1" library_urn="urn:adsk.eagle:library:371" deviceset="+3V3" device=""/>
-<part name="GND6" library="supply1" library_urn="urn:adsk.eagle:library:371" deviceset="GND" device=""/>
-<part name="C1" library="SIG_Parts" deviceset="CAP_CERAMIC_*" device="0402"/>
-<part name="+3V7" library="supply1" library_urn="urn:adsk.eagle:library:371" deviceset="+3V3" device=""/>
-<part name="GND7" library="supply1" library_urn="urn:adsk.eagle:library:371" deviceset="GND" device=""/>
-<part name="JP4" library="SparkFun-Jumpers" library_urn="urn:adsk.eagle:library:528" deviceset="JUMPER-SMT_2_NO" device="_NO-SILK" package3d_urn="urn:adsk.eagle:package:39277/1" value="AL0"/>
-<part name="JP5" library="SparkFun-Jumpers" library_urn="urn:adsk.eagle:library:528" deviceset="JUMPER-SMT_2_NO" device="_NO-SILK" package3d_urn="urn:adsk.eagle:package:39277/1" value="AL1"/>
-<part name="JP6" library="SparkFun-Jumpers" library_urn="urn:adsk.eagle:library:528" deviceset="JUMPER-SMT_2_NO" device="_NO-SILK" package3d_urn="urn:adsk.eagle:package:39277/1" value="AL2"/>
-<part name="JP7" library="SparkFun-Jumpers" library_urn="urn:adsk.eagle:library:528" deviceset="JUMPER-SMT_2_NO" device="_NO-SILK" package3d_urn="urn:adsk.eagle:package:39277/1" value="AL3"/>
-<part name="JP8" library="SparkFun-Jumpers" library_urn="urn:adsk.eagle:library:528" deviceset="JUMPER-SMT_2_NO" device="_NO-SILK" package3d_urn="urn:adsk.eagle:package:39277/1" value="AL4"/>
-<part name="X2" library="SIG_Parts" deviceset="FFC_10P" device="V">
+<part name="IC1" library="temp_sens_ring" library_urn="urn:adsk.eagle:library:31797301" deviceset="MCP9808" device="" package3d_urn="urn:adsk.eagle:package:31797270/2"/>
+<part name="+3V1" library="temp_sens_ring" library_urn="urn:adsk.eagle:library:31797301" deviceset="+3V3" device=""/>
+<part name="+3V2" library="temp_sens_ring" library_urn="urn:adsk.eagle:library:31797301" deviceset="+3V3" device=""/>
+<part name="+3V3" library="temp_sens_ring" library_urn="urn:adsk.eagle:library:31797301" deviceset="+3V3" device=""/>
+<part name="GND1" library="temp_sens_ring" library_urn="urn:adsk.eagle:library:31797301" deviceset="GND" device=""/>
+<part name="GND2" library="temp_sens_ring" library_urn="urn:adsk.eagle:library:31797301" deviceset="GND" device=""/>
+<part name="GND3" library="temp_sens_ring" library_urn="urn:adsk.eagle:library:31797301" deviceset="GND" device=""/>
+<part name="GND4" library="temp_sens_ring" library_urn="urn:adsk.eagle:library:31797301" deviceset="GND" device=""/>
+<part name="+3V4" library="temp_sens_ring" library_urn="urn:adsk.eagle:library:31797301" deviceset="+3V3" device=""/>
+<part name="R1" library="temp_sens_ring" library_urn="urn:adsk.eagle:library:31797301" deviceset="RESISTOR_*" device="0402" package3d_urn="urn:adsk.eagle:package:31797273/2" value="10K"/>
+<part name="+3V5" library="temp_sens_ring" library_urn="urn:adsk.eagle:library:31797301" deviceset="+3V3" device=""/>
+<part name="GND5" library="temp_sens_ring" library_urn="urn:adsk.eagle:library:31797301" deviceset="GND" device=""/>
+<part name="+3V6" library="temp_sens_ring" library_urn="urn:adsk.eagle:library:31797301" deviceset="+3V3" device=""/>
+<part name="GND6" library="temp_sens_ring" library_urn="urn:adsk.eagle:library:31797301" deviceset="GND" device=""/>
+<part name="C1" library="temp_sens_ring" library_urn="urn:adsk.eagle:library:31797301" deviceset="CAP_CERAMIC_*" device="0402" package3d_urn="urn:adsk.eagle:package:31797388/2"/>
+<part name="+3V7" library="temp_sens_ring" library_urn="urn:adsk.eagle:library:31797301" deviceset="+3V3" device=""/>
+<part name="GND7" library="temp_sens_ring" library_urn="urn:adsk.eagle:library:31797301" deviceset="GND" device=""/>
+<part name="JP4" library="temp_sens_ring" library_urn="urn:adsk.eagle:library:31797301" deviceset="JUMPER-SMT_2_NO" device="_NO-SILK" package3d_urn="urn:adsk.eagle:package:31797260/2" value="AL0"/>
+<part name="JP5" library="temp_sens_ring" library_urn="urn:adsk.eagle:library:31797301" deviceset="JUMPER-SMT_2_NO" device="_NO-SILK" package3d_urn="urn:adsk.eagle:package:31797260/2" value="AL1"/>
+<part name="JP6" library="temp_sens_ring" library_urn="urn:adsk.eagle:library:31797301" deviceset="JUMPER-SMT_2_NO" device="_NO-SILK" package3d_urn="urn:adsk.eagle:package:31797260/2" value="AL2"/>
+<part name="JP7" library="temp_sens_ring" library_urn="urn:adsk.eagle:library:31797301" deviceset="JUMPER-SMT_2_NO" device="_NO-SILK" package3d_urn="urn:adsk.eagle:package:31797260/2" value="AL3"/>
+<part name="JP8" library="temp_sens_ring" library_urn="urn:adsk.eagle:library:31797301" deviceset="JUMPER-SMT_2_NO" device="_NO-SILK" package3d_urn="urn:adsk.eagle:package:31797260/2" value="AL4"/>
+<part name="X2" library="temp_sens_ring" library_urn="urn:adsk.eagle:library:31797301" deviceset="FFC_10P" device="V" package3d_urn="urn:adsk.eagle:package:31797271/2">
 <attribute name="MFR" value="XFCN"/>
 <attribute name="MFR_PART" value="F1002-B-10-20T-R"/>
 <attribute name="PITCH" value="1.00"/>
 </part>
-<part name="GND8" library="supply1" library_urn="urn:adsk.eagle:library:371" deviceset="GND" device=""/>
-<part name="GND9" library="supply1" library_urn="urn:adsk.eagle:library:371" deviceset="GND" device=""/>
-<part name="+3V8" library="supply1" library_urn="urn:adsk.eagle:library:371" deviceset="+3V3" device=""/>
-<part name="J2" library="SIG_Parts" deviceset="SMD_JUMP_2_NO_" device="S"/>
-<part name="J1" library="SIG_Parts" deviceset="SMD_JUMP_2_NO_" device="S"/>
-<part name="J3" library="SIG_Parts" deviceset="SMD_JUMP_2_NO_" device="S"/>
-<part name="GND10" library="supply1" library_urn="urn:adsk.eagle:library:371" deviceset="GND" device=""/>
-<part name="R2" library="SIG_Parts" deviceset="RESISTOR_NET_*" device="4-0502"/>
-<part name="FRAME1" library="SIG_Parts" deviceset="FRAME_A4_FULL" device=""/>
+<part name="GND8" library="temp_sens_ring" library_urn="urn:adsk.eagle:library:31797301" deviceset="GND" device=""/>
+<part name="GND9" library="temp_sens_ring" library_urn="urn:adsk.eagle:library:31797301" deviceset="GND" device=""/>
+<part name="+3V8" library="temp_sens_ring" library_urn="urn:adsk.eagle:library:31797301" deviceset="+3V3" device=""/>
+<part name="J2" library="temp_sens_ring" library_urn="urn:adsk.eagle:library:31797301" deviceset="SMD_JUMP_2_NO_" device="S" package3d_urn="urn:adsk.eagle:package:31797261/2"/>
+<part name="J1" library="temp_sens_ring" library_urn="urn:adsk.eagle:library:31797301" deviceset="SMD_JUMP_2_NO_" device="S" package3d_urn="urn:adsk.eagle:package:31797261/2"/>
+<part name="J3" library="temp_sens_ring" library_urn="urn:adsk.eagle:library:31797301" deviceset="SMD_JUMP_2_NO_" device="S" package3d_urn="urn:adsk.eagle:package:31797261/2"/>
+<part name="GND10" library="temp_sens_ring" library_urn="urn:adsk.eagle:library:31797301" deviceset="GND" device=""/>
+<part name="R2" library="temp_sens_ring" library_urn="urn:adsk.eagle:library:31797301" deviceset="RESISTOR_NET_*" device="4-0502" package3d_urn="urn:adsk.eagle:package:31797268/2"/>
+<part name="FRAME1" library="temp_sens_ring" library_urn="urn:adsk.eagle:library:31797301" deviceset="FRAME_A4_FULL" device=""/>
 </parts>
 <sheets>
