File: hardware/RAK3172_board/RAK3172_board.brd (EAGLE design)
At the start: 58 x 30 mm, 45 parts, among them IC1 LTC4311, IC2 RAK3172HF, Q1 BSS138, Q2 BSS84, X1 PWR, X2 GPIO, X3 UART, X4 JTAG, X5 PROG, X6 I2C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

Commit message: Latest hardware designs
Parts:
- R6, R7: value (none) -> 2.2K
Changed lines of the file:
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@@
 <layer number="14" name="Route14" color="22" fill="1" visible="no" active="no"/>
 <layer number="15" name="Route15" color="23" fill="1" visible="no" active="no"/>
-<layer number="16" name="Bottom" color="1" fill="1" visible="no" active="yes"/>
+<layer number="16" name="Bottom" color="1" fill="1" visible="yes" active="yes"/>
 <layer number="17" name="Pads" color="2" fill="1" visible="yes" active="yes"/>
 <layer number="18" name="Vias" color="2" fill="1" visible="yes" active="yes"/>
@@
 <attribute name="NAME" x="31.21" y="0.933" size="0.6096" layer="26" font="vector" ratio="20" rot="MR0" align="bottom-center"/>
 </element>
-<element name="R6" library="RAK3172_board" library_urn="urn:adsk.eagle:library:32884481" package="SMD_0603" package3d_urn="urn:adsk.eagle:package:32884545/2" value="" x="39.17" y="3.74" smashed="yes">
+<element name="R6" library="RAK3172_board" library_urn="urn:adsk.eagle:library:32884481" package="SMD_0603" package3d_urn="urn:adsk.eagle:package:32884545/2" value="2.2K" x="39.17" y="3.74" smashed="yes">
 <attribute name="NAME" x="40.885" y="3.375" size="0.8" layer="25" font="vector" ratio="15"/>
 <attribute name="VALUE" x="37.365" y="2.285" size="0.5" layer="27" font="vector" ratio="15" rot="R90"/>
 </element>
-<element name="R7" library="RAK3172_board" library_urn="urn:adsk.eagle:library:32884481" package="SMD_0603" package3d_urn="urn:adsk.eagle:package:32884545/2" value="" x="39.17" y="2.16" smashed="yes">
+<element name="R7" library="RAK3172_board" library_urn="urn:adsk.eagle:library:32884481" package="SMD_0603" package3d_urn="urn:adsk.eagle:package:32884545/2" value="2.2K" x="39.17" y="2.16" smashed="yes">
 <attribute name="NAME" x="40.885" y="1.845" size="0.8" layer="25" font="vector" ratio="15"/>
 </element>
