File: hardware/RAK3172_board/RAK3172_board.sch (EAGLE design)
At the start: 44 parts, among them IC1 LTC4311, IC2 RAK3172HF, Q1 BSS138, Q2 BSS84, X1 PWR, X2 GPIO, X3 UART, X4 JTAG, X5 PROG, X6 I2C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

Commit message: Latest hardware designs
Parts:
- R6, R7: value (none) -> 2.2K
Changed lines of the file:
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@@
 <part name="JP1" library="RAK3172_board" library_urn="urn:adsk.eagle:library:32884481" deviceset="JUMPER-SMT_3_1-NC_PASTE" device="_SILK" package3d_urn="urn:adsk.eagle:package:32884565/2"/>
 <part name="+3.3V_10" library="RAK3172_board" library_urn="urn:adsk.eagle:library:32884481" deviceset="+3.3V" device=""/>
-<part name="R6" library="RAK3172_board" library_urn="urn:adsk.eagle:library:32884481" deviceset="RESISTOR_*" device="0603" package3d_urn="urn:adsk.eagle:package:32884545/2"/>
-<part name="R7" library="RAK3172_board" library_urn="urn:adsk.eagle:library:32884481" deviceset="RESISTOR_*" device="0603" package3d_urn="urn:adsk.eagle:package:32884545/2"/>
+<part name="R6" library="RAK3172_board" library_urn="urn:adsk.eagle:library:32884481" deviceset="RESISTOR_*" device="0603" package3d_urn="urn:adsk.eagle:package:32884545/2" value="2.2K"/>
+<part name="R7" library="RAK3172_board" library_urn="urn:adsk.eagle:library:32884481" deviceset="RESISTOR_*" device="0603" package3d_urn="urn:adsk.eagle:package:32884545/2" value="2.2K"/>
 <part name="+3.3V_11" library="RAK3172_board" library_urn="urn:adsk.eagle:library:32884481" deviceset="+3.3V" device=""/>
 <part name="+3.3V_12" library="RAK3172_board" library_urn="urn:adsk.eagle:library:32884481" deviceset="+3.3V" device=""/>
